Commit message: update files setup

File: genesis_playground/resources/zbot/robot_fixed.urdf (robot description, URDF)
Before this commit: robot z-bot2_fe_urdf, 20 links, 19 joints
Joints:
- joint L_Ankle_Pitch: limit lower=-0.9 upper=0.9 effort=1.91 velocity=10 -> lower=-0.9 upper=0.9 effort=10 velocity=10
- joint L_Hip_Pitch: limit lower=-1.54 upper=1.0 effort=1.91 velocity=10 -> lower=-1.54 upper=1.0 effort=10 velocity=10
- joint L_Hip_Roll: limit lower=-0.7 upper=0.7 effort=1.91 velocity=10 -> lower=-0.7 upper=0.7 effort=10 velocity=10
- joint L_Hip_Yaw: limit lower=-1.54 upper=0.157 effort=1.91 velocity=10 -> lower=-0.3 upper=0.157 effort=10 velocity=10
- joint L_Knee_Pitch: limit lower=0 upper=1.57 effort=1.91 velocity=10 -> lower=0 upper=1.57 effort=10 velocity=10
- joint R_Ankle_Pitch: limit lower=-0.9 upper=0.9 effort=1.91 velocity=10 -> lower=-0.9 upper=0.9 effort=10 velocity=10
- joint R_Hip_Pitch: limit lower=-1.0 upper=1.54 effort=1.91 velocity=10 -> lower=-1.0 upper=1.54 effort=10 velocity=10
- joint R_Hip_Roll: limit lower=-0.7 upper=0.7 effort=1.91 velocity=10 -> lower=-0.7 upper=0.7 effort=10 velocity=10
- joint R_Hip_Yaw: limit lower=-1.54 upper=0.157 effort=1.91 velocity=10 -> lower=-0.3 upper=0.157 effort=10 velocity=10
- joint R_Knee_Pitch: limit lower=-1.57 upper=0 effort=1.91 velocity=10 -> lower=-1.57 upper=0 effort=10 velocity=10
