Commit message: trying to change to new urdf + some small debugs

File: genesis_playground/resources/zbot/robot_fixed_noisy_0.urdf (robot description, URDF)
Before this commit: robot z-bot2_fe_urdf, 20 links, 19 joints
Links:
- link FOOT: mass 0.32814002999999997 -> 0.3566673917021253
- link FOOT_2: mass 0.32814002999999997 -> 0.3307809076535634
- link Z-BOT2_MASTER-BODY-SKELETON: mass 1.5982792056799995 -> 1.5339120884741244

File: genesis_playground/resources/zbot/robot_fixed_noisy_1.urdf (robot description, URDF)
Before this commit: robot z-bot2_fe_urdf, 20 links, 19 joints
Links:
- link FOOT: mass 0.32814002999999997 -> 0.23438946333881094
- link FOOT_2: mass 0.32814002999999997 -> 0.27791222894778084
- link Z-BOT2_MASTER-BODY-SKELETON: mass 1.5982792056799995 -> 1.5547087922635867

File: genesis_playground/resources/zbot/robot_fixed_noisy_10.urdf (robot description, URDF)
Before this commit: robot z-bot2_fe_urdf, 20 links, 19 joints
Links:
- link FOOT: mass 0.32814002999999997 -> 0.23029442540438186
- link FOOT_2: mass 0.32814002999999997 -> 0.25654620826425195
- link Z-BOT2_MASTER-BODY-SKELETON: mass 1.5982792056799995 -> 1.5429728384282981

File: genesis_playground/resources/zbot/robot_fixed_noisy_11.urdf (robot description, URDF)
Before this commit: robot z-bot2_fe_urdf, 20 links, 19 joints
Links:
- link FOOT: mass 0.32814002999999997 -> 0.28545870237952586
- link FOOT_2: mass 0.32814002999999997 -> 0.28775544028401734
- link Z-BOT2_MASTER-BODY-SKELETON: mass 1.5982792056799995 -> 1.5447912843317424

File: genesis_playground/resources/zbot/robot_fixed_noisy_12.urdf (robot description, URDF)
Before this commit: robot z-bot2_fe_urdf, 20 links, 19 joints
Links:
- link FOOT: mass 0.32814002999999997 -> 0.28810281578266467
- link FOOT_2: mass 0.32814002999999997 -> 0.19386598593222776
- link Z-BOT2_MASTER-BODY-SKELETON: mass 1.5982792056799995 -> 1.4877710556182113

File: genesis_playground/resources/zbot/robot_fixed_noisy_13.urdf (robot description, URDF)
Before this commit: robot z-bot2_fe_urdf, 20 links, 19 joints
Links:
- link FOOT: mass 0.32814002999999997 -> 0.3130621974794307
- link FOOT_2: mass 0.32814002999999997 -> 0.3137318688619128
- link Z-BOT2_MASTER-BODY-SKELETON: mass 1.5982792056799995 -> 1.4990027549154878

File: genesis_playground/resources/zbot/robot_fixed_noisy_14.urdf (robot description, URDF)
Before this commit: robot z-bot2_fe_urdf, 20 links, 19 joints
Links:
- link FOOT: mass 0.32814002999999997 -> 0.339486908793846
- link FOOT_2: mass 0.32814002999999997 -> 0.3482846084765925
- link Z-BOT2_MASTER-BODY-SKELETON: mass 1.5982792056799995 -> 1.444741357962369

File: genesis_playground/resources/zbot/robot_fixed_noisy_15.urdf (robot description, URDF)
Before this commit: robot z-bot2_fe_urdf, 20 links, 19 joints
Links:
- link FOOT: mass 0.32814002999999997 -> 0.376692598704804
- link FOOT_2: mass 0.32814002999999997 -> 0.30214838592970783
- link Z-BOT2_MASTER-BODY-SKELETON: mass 1.5982792056799995 -> 1.4700194652847594

File: genesis_playground/resources/zbot/robot_fixed_noisy_16.urdf (robot description, URDF)
Before this commit: robot z-bot2_fe_urdf, 20 links, 19 joints
Links:
- link FOOT: mass 0.32814002999999997 -> 0.27179391344751114
- link FOOT_2: mass 0.32814002999999997 -> 0.2096682719577863
- link Z-BOT2_MASTER-BODY-SKELETON: mass 1.5982792056799995 -> 1.5409214880242517

File: genesis_playground/resources/zbot/robot_fixed_noisy_17.urdf (robot description, URDF)
Before this commit: robot z-bot2_fe_urdf, 20 links, 19 joints
Links:
- link FOOT: mass 0.32814002999999997 -> 0.20492514294536354
- link FOOT_2: mass 0.32814002999999997 -> 0.27190963722094713
- link Z-BOT2_MASTER-BODY-SKELETON: mass 1.5982792056799995 -> 1.5726030467547796

File: genesis_playground/resources/zbot/robot_fixed_noisy_18.urdf (robot description, URDF)
Before this commit: robot z-bot2_fe_urdf, 20 links, 19 joints
Links:
- link FOOT: mass 0.32814002999999997 -> 0.3373688880151273
- link FOOT_2: mass 0.32814002999999997 -> 0.17463888297857671
- link Z-BOT2_MASTER-BODY-SKELETON: mass 1.5982792056799995 -> 1.4762437237983606

File: genesis_playground/resources/zbot/robot_fixed_noisy_19.urdf (robot description, URDF)
Before this commit: robot z-bot2_fe_urdf, 20 links, 19 joints
Links:
- link FOOT: mass 0.32814002999999997 -> 0.31650754348304133
- link FOOT_2: mass 0.32814002999999997 -> 0.29263509967122975
- link Z-BOT2_MASTER-BODY-SKELETON: mass 1.5982792056799995 -> 1.5553014151758935

File: genesis_playground/resources/zbot/robot_fixed_noisy_2.urdf (robot description, URDF)
Before this commit: robot z-bot2_fe_urdf, 20 links, 19 joints
Links:
- link FOOT: mass 0.32814002999999997 -> 0.3003332125223721
- link FOOT_2: mass 0.32814002999999997 -> 0.24149471629767788
- link Z-BOT2_MASTER-BODY-SKELETON: mass 1.5982792056799995 -> 1.530351891431863

File: genesis_playground/resources/zbot/robot_fixed_noisy_3.urdf (robot description, URDF)
Before this commit: robot z-bot2_fe_urdf, 20 links, 19 joints
Links:
- link FOOT: mass 0.32814002999999997 -> 0.21200671534037524
- link FOOT_2: mass 0.32814002999999997 -> 0.15047420810237858
- link Z-BOT2_MASTER-BODY-SKELETON: mass 1.5982792056799995 -> 1.5708683618121084

File: genesis_playground/resources/zbot/robot_fixed_noisy_4.urdf (robot description, URDF)
Before this commit: robot z-bot2_fe_urdf, 20 links, 19 joints
Links:
- link FOOT: mass 0.32814002999999997 -> 0.3451031622552299
- link FOOT_2: mass 0.32814002999999997 -> 0.32958508451304036
- link Z-BOT2_MASTER-BODY-SKELETON: mass 1.5982792056799995 -> 1.5266965891308797

File: genesis_playground/resources/zbot/robot_fixed_noisy_5.urdf (robot description, URDF)
Before this commit: robot z-bot2_fe_urdf, 20 links, 19 joints
Links:
- link FOOT: mass 0.32814002999999997 -> 0.1940471870154709
- link FOOT_2: mass 0.32814002999999997 -> 0.276011540591062
- link Z-BOT2_MASTER-BODY-SKELETON: mass 1.5982792056799995 -> 1.5083988614200112

File: genesis_playground/resources/zbot/robot_fixed_noisy_6.urdf (robot description, URDF)
Before this commit: robot z-bot2_fe_urdf, 20 links, 19 joints
Links:
- link FOOT: mass 0.32814002999999997 -> 0.29528970982915037
- link FOOT_2: mass 0.32814002999999997 -> 0.34069577276413476
- link Z-BOT2_MASTER-BODY-SKELETON: mass 1.5982792056799995 -> 1.5509424786402344

File: genesis_playground/resources/zbot/robot_fixed_noisy_7.urdf (robot description, URDF)
Before this commit: robot z-bot2_fe_urdf, 20 links, 19 joints
Links:
- link FOOT: mass 0.32814002999999997 -> 0.3264237220920659
- link FOOT_2: mass 0.32814002999999997 -> 0.2245897502001849
- link Z-BOT2_MASTER-BODY-SKELETON: mass 1.5982792056799995 -> 1.6084785670182775

File: genesis_playground/resources/zbot/robot_fixed_noisy_8.urdf (robot description, URDF)
Before this commit: robot z-bot2_fe_urdf, 20 links, 19 joints
Links:
- link FOOT: mass 0.32814002999999997 -> 0.22504727063226748
- link FOOT_2: mass 0.32814002999999997 -> 0.27469930777724183
- link Z-BOT2_MASTER-BODY-SKELETON: mass 1.5982792056799995 -> 1.5812009148796702

File: genesis_playground/resources/zbot/robot_fixed_noisy_9.urdf (robot description, URDF)
Before this commit: robot z-bot2_fe_urdf, 20 links, 19 joints
Links:
- link FOOT: mass 0.32814002999999997 -> 0.27404252984042515
- link FOOT_2: mass 0.32814002999999997 -> 0.3985641198407805
- link Z-BOT2_MASTER-BODY-SKELETON: mass 1.5982792056799995 -> 1.5939496838157075
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